Commit message: Please enter the commit message for your changes. Lines starting with '#' will be ignored, and an empty message aborts the commit.
HEAD detached from f906de7
Changes to be committed:
	new file:   tm_description/urdf/tm5-700.srdf
	new file:   tm_description/urdf/tm5700.urdf
	deleted:    tm_description/xacro/macro.tm5-700-nominal2.urdf.xacro
	new file:   tm_description/xacro/tm5-700.ros2_control.xacro
	new file:   tm_description/xacro/tm5-700.srdf
	modified:   tm_description/xacro/tm5-700.urdf.xacro
	new file:   tm_description/xacro/tm5700.urdf
	new file:   tm_moveit_config_tm5-700/config/initial_positions.yaml
	modified:   tm_moveit_config_tm5-700/config/joint_limits.yaml
	modified:   tm_moveit_config_tm5-700/config/kinematics.yaml
	new file:   tm_moveit_config_tm5-700/config/moveit_controllers.yaml
	new file:   tm_moveit_config_tm5-700/config/pilz_cartesian_limits.yaml
	new file:   tm_moveit_config_tm5-700/config/ros2_controllers.yaml
	new file:   tm_moveit_config_tm5-700/config/ros_controllers (copy).yaml
	modified:   tm_moveit_config_tm5-700/config/ros_controllers.yaml
	modified:   tm_moveit_config_tm5-700/config/tm5-700.srdf
	modified:   tm_moveit_cpp_demo/config/controllers.yaml
	modified:   tm_moveit_cpp_demo/launch/tm5-700_run_moveit_cpp.launch.py
	modified:   tm_moveit_cpp_demo/src/run_moveit_cpp.cpp

File: tm_description/xacro/tm5-700.urdf.xacro (robot description, xacro)
@@ -1,27 +1,9 @@
 <?xml version="1.0"?>
 <robot xmlns:xacro="http://www.ros.org/wiki/xacro" name="tm5-700">
-  <xacro:arg name="ns" default="" />
-  <xacro:arg name="prefix" default="" />
-  <xacro:arg name="color" default="none" />
-  <xacro:arg name="trans_hw_iface" default="hardware_interface/PositionJointInterface" />
-  <xacro:include filename="$(find tm_description)/xacro/macro.gazebo.xacro" />
-  <xacro:include filename="$(find tm_description)/xacro/macro.transmission.xacro" />
-  <xacro:include filename="$(find tm_description)/xacro/macro.materials.xacro" />
-  <!-- tm5-700 -->
-  <!-- If the user want to use newly generated named robot description file as user_defined.urdf.xacro, -->
-  <!-- you must modify 'macro.tm5-700-nominal.urdf.xacro' to 'user_defined.urdf.xacro'  -->
-  <xacro:include filename="$(find tm_description)/xacro/macro.tm5-700-nominal.urdf.xacro" />
-  <!--  -->
-  <xacro:tmr_gazebo ns="$(arg ns)" prefix="$(arg prefix)" />
-  <xacro:tmr_transmission prefix="$(arg prefix)" hw_iface="$(arg trans_hw_iface)" />
-  <xacro:tmr_materials/>
-  <!-- Arm -->
-  <xacro:property name="color" value="$(arg color)"/>
-  <xacro:if value="${color == 'none'}">
-    <xacro:tm5-700 ns="$(arg ns)" prefix="$(arg prefix)" />
-  </xacro:if>
-  <!-- Arm.color.stl -->
-  <xacro:unless value="${color == 'none'}">
-    <xacro:tm5-700 ns="$(arg ns)" prefix="$(arg prefix)" color="${color}" format="stl" />
-  </xacro:unless>
+    <xacro:arg name="initial_positions_file" default="initial_positions.yaml" />
+    <!-- Import tm5-700 urdf file -->
+    <xacro:include filename="$(find tm_description)/xacro/tm5700.urdf" />
+    <!-- Import control_xacro -->
+    <xacro:include filename="tm5-700.ros2_control.xacro" />
+    <xacro:tm5-700_ros2_control name="FakeSystem" initial_positions_file="$(arg initial_positions_file)"/>
 </robot>

Commit message: modified:   tm_description/xacro/tm5-700.urdf.xacro 	modified:   tm_moveit_cpp_demo/launch/tm5-700_run_moveit_cpp.launch.py

File: tm_description/xacro/tm5-700.urdf.xacro (robot description, xacro)
@@ -1,9 +1,45 @@
 <?xml version="1.0"?>
 <robot xmlns:xacro="http://www.ros.org/wiki/xacro" name="tm5-700">
-    <xacro:arg name="initial_positions_file" default="initial_positions.yaml" />
-    <!-- Import tm5-700 urdf file -->
-    <xacro:include filename="$(find tm_description)/xacro/tm5700.urdf" />
-    <!-- Import control_xacro -->
-    <xacro:include filename="tm5-700.ros2_control.xacro" />
-    <xacro:tm5-700_ros2_control name="FakeSystem" initial_positions_file="$(arg initial_positions_file)"/>
+  <xacro:arg name="ns" default="" />
+  <xacro:arg name="prefix" default="" />
+  <xacro:arg name="color" default="none" />
+  <xacro:arg name="trans_hw_iface" default="hardware_interface/PositionJointInterface" />
+  <xacro:include filename="$(find tm_description)/xacro/macro.gazebo.xacro" />
+  <xacro:include filename="$(find tm_description)/xacro/macro.transmission.xacro" />
+  <xacro:include filename="$(find tm_description)/xacro/macro.materials.xacro" />
+  <!-- tm5-700 -->
+  <!-- If the user want to use newly generated named robot description file as user_defined.urdf.xacro, -->
+  <!-- you must modify 'macro.tm5-700-nominal.urdf.xacro' to 'user_defined.urdf.xacro'  -->
+  <xacro:include filename="$(find tm_description)/xacro/macro.tm5-700-nominal.urdf.xacro" />
+  <!--  -->
+  <xacro:tmr_gazebo ns="$(arg ns)" prefix="$(arg prefix)" />
+  <xacro:tmr_transmission prefix="$(arg prefix)" hw_iface="$(arg trans_hw_iface)" />
+  <xacro:tmr_materials/>
+  <!-- Arm -->
+  <xacro:property name="color" value="$(arg color)"/>
+  <xacro:if value="${color == 'none'}">
+    <xacro:tm5-700 ns="$(arg ns)" prefix="left" />
+  </xacro:if>
+  <xacro:property name="color" value="$(arg color)"/>
+  <xacro:if value="${color == 'none'}">
+    <xacro:tm5-700 ns="$(arg ns)" prefix="right" />
+  </xacro:if>
+  <!-- Arm.color.stl -->
+  <xacro:unless value="${color == 'none'}">
+    <xacro:tm5-700 ns="$(arg ns)" prefix="left" color="${color}" format="stl" />
+  </xacro:unless>
+  <xacro:unless value="${color == 'none'}">
+    <xacro:tm5-700 ns="$(arg ns)" prefix="right" color="${color}" format="stl" />
+  </xacro:unless>
+  <link name="base"/>
+  <joint name="base_to_left" type="fixed">
+    <parent link="base"/>
+    <child link="leftbase"/>
+    <origin rpy="0.000000 0.000000 0.000000" xyz="0.000000 0.000000 0.000000"/>
+  </joint>
+  <joint name="base_to_right" type="fixed">
+    <parent link="base"/>
+    <child link="rightbase"/>
+    <origin rpy="0.000000 0.000000 0.000000" xyz="0.000000 1.200000 0.000000"/>
+  </joint>
 </robot>

Commit message: new file:   tm_description/meshes/hanoi/base.stl 	new file:   tm_description/meshes/hanoi/peca_amarela_1.stl 	new file:   tm_description/meshes/hanoi/peca_amarela_2.stl 	new file:   tm_description/meshes/hanoi/peca_amarela_3.stl 	new file:   tm_description/meshes/hanoi/peca_azul_1.stl 	new file:   tm_description/meshes/hanoi/peca_azul_2.stl 	new file:   tm_description/meshes/hanoi/peca_azul_3.stl 	new file:   tm_description/meshes/hanoi/peca_verde_1.stl 	new file:   tm_description/meshes/hanoi/peca_verde_2.stl 	new file:   tm_description/meshes/hanoi/peca_verde_3.stl 	new file:   tm_description/meshes/hanoi/peca_vermelha_1.stl 	new file:   tm_description/meshes/hanoi/peca_vermelha_2.stl 	new file:   tm_description/meshes/hanoi/peca_vermelha_3.stl 	new file:   tm_description/meshes/hanoi/table.stl 	modified:   tm_description/xacro/tm5-700.urdf.xacro 	modified:   tm_moveit_cpp_demo/src/run_moveit_cpp.cpp

File: tm_description/xacro/tm5-700.urdf.xacro (robot description, xacro)
@@ -41,5 +41,129 @@
     <parent link="base"/>
     <child link="rightbase"/>
-    <origin rpy="0.000000 0.000000 0.000000" xyz="0.000000 1.200000 0.000000"/>
+    <origin rpy="0.000000 0.000000 0.000000" xyz="0.000000 1.175000 0.000000"/>
+  </joint>
+  <!-- TORRE DE HANOI -->
+  <link name="hanoi_base">
+    <visual>
+      <origin xyz="-0.058 -0.044 -0.01" rpy="0 0 0" />
+      <geometry>
+        <mesh filename="package://tm_description/meshes/hanoi/base.stl" scale="0.001 0.001 0.001"/>
+      </geometry>
+      <material name="Color_hbase">
+        <color rgba="0.643 0.454 0.286 1"/>
+      </material>
+    </visual>
+  </link>
+  <!-- arrumar medidas do robo esq para pino1 da torre -->
+  <joint name="Jmesa" type="fixed">
+    <origin xyz="0.3 0.4 0" rpy="0 0 1.57" />
+    <parent link="base"/>
+    <child link="hanoi_base"/>
+  </joint>
+  <joint name="Jp1" type="prismatic">
+    <origin xyz="0 0 0" rpy="0 0 0" />
+    <limit effort="30" velocity="1.0" lower="-2.2" upper="0.7" />
+    <parent link="hanoi_base"/>
+    <child link="hanoi_p1"/>
+  </joint>
+  <link name="hanoi_p1">
+    <visual>
+      <origin xyz="0 0 0" rpy="0 0 0" />
+      <geometry>
+        <mesh filename="package://tm_description/meshes/hanoi/peca_vermelha_1.stl" scale="0.001 0.001 0.001"/>
+      </geometry>
+      <!--material name="Peca_amarela">
+        <color rgba="1 0.788 0.121 1"/-->
+      <!--material name="Peca_azul">
+        <color rgba="0 0.352 0.580 1"/-->
+      <material name="Peca_vermelha">
+        <color rgba="0.901 0.168 0.156 1"/>
+      </material>
+    </visual>
+  </link>
+  <link name="hanoi_p2">
+    <visual>
+      <origin xyz="0 0 0" rpy="0 0 0" />
+      <geometry>
+        <mesh filename="package://tm_description/meshes/hanoi/peca_vermelha_2.stl" scale="0.001 0.001 0.001"/>
+      </geometry>
+      <material name="Peca_vermelha">
+        <color rgba="0.901 0.168 0.156 1"/>
+      </material>
+    </visual>
+  </link>
+  <joint name="Jp2" type="prismatic">
+    <origin xyz="0 0 0.013" rpy="0 0 0" />
+    <limit effort="30" velocity="1.0" lower="-2.2" upper="0.7" />
+    <parent link="hanoi_base"/>
+    <child link="hanoi_p2"/>
+  </joint>
+  <link name="hanoi_p3">
+    <visual>
+      <origin xyz="0 0 0" rpy="0 0 0" />
+      <geometry>
+        <mesh filename="package://tm_description/meshes/hanoi/peca_vermelha_3.stl" scale="0.001 0.001 0.001"/>
+      </geometry>
+      <material name="Peca_vermelha">
+        <color rgba="0.901 0.168 0.156 1"/>
+      </material>
+    </visual>
+  </link>
+  <joint name="Jp3" type="prismatic">
+    <origin xyz="0 0 0.026" rpy="0 0 0" />
+    <limit effort="30" velocity="1.0" lower="-2.2" upper="0.7" />
+    <parent link="hanoi_base"/>
+    <child link="hanoi_p3"/>
+  </joint>
+  <link name="hanoi_p4">
+    <visual>
+      <origin xyz="0 0 0" rpy="0 0 0" />
+      <geometry>
+        <mesh filename="package://tm_description/meshes/hanoi/peca_verde_1.stl" scale="0.001 0.001 0.001"/>
+      </geometry>
+      <material name="Peca_verde">
+        <color rgba="0.670 0.858 0.160 1"/>
+      </material>
+    </visual>
+  </link>
+  <joint name="Jp4" type="prismatic">
+    <origin xyz="0.088 0 0" rpy="0 0 0" />
+    <limit effort="30" velocity="1.0" lower="-2.2" upper="0.7" />
+    <parent link="hanoi_base"/>
+    <child link="hanoi_p4"/>
+  </joint>
+  <link name="hanoi_p5">
+    <visual>
+      <origin xyz="0 0 0" rpy="0 0 0" />
+      <geometry>
+        <mesh filename="package://tm_description/meshes/hanoi/peca_verde_2.stl" scale="0.001 0.001 0.001"/>
+      </geometry>
+      <material name="Peca_verde">
+        <color rgba="0.670 0.858 0.160 1"/>
+      </material>
+    </visual>
+  </link>
+  <joint name="Jp5" type="prismatic">
+    <origin xyz="0.088 0 0.013" rpy="0 0 0" />
+    <limit effort="30" velocity="1.0" lower="-2.2" upper="0.7" />
+    <parent link="hanoi_base"/>
+    <child link="hanoi_p5"/>
+  </joint>
+  <link name="hanoi_p6">
+    <visual>
+      <origin xyz="0 0 0" rpy="0 0 0" />
+      <geometry>
+        <mesh filename="package://tm_description/meshes/hanoi/peca_verde_3.stl" scale="0.001 0.001 0.001"/>
+      </geometry>
+      <material name="Peca_verde">
+        <color rgba="0.670 0.858 0.160 1"/>
+      </material>
+    </visual>
+  </link>
+  <joint name="Jp6" type="prismatic">
+    <origin xyz="0.088 0 0.026" rpy="0 0 0" />
+    <limit effort="30" velocity="1.0" lower="-2.2" upper="0.7" />
+    <parent link="hanoi_base"/>
+    <child link="hanoi_p6"/>
   </joint>
 </robot>

Commit message: modified:   Comandos.txt 	new file:   tm_description/xacro/hanoi.xacro 	modified:   tm_description/xacro/tm5-700.urdf.xacro

File: tm_description/xacro/tm5-700.urdf.xacro (robot description, xacro)
@@ -25,4 +25,6 @@
     <xacro:tm5-700 ns="$(arg ns)" prefix="right" />
   </xacro:if>
+  <xacro:tm5-700 ns="$(arg ns)" prefix="left1" color="green" format="stl"/>
+  <xacro:tm5-700 ns="$(arg ns)" prefix="right1" color="green" format="stl"/>
   <!-- Arm.color.stl -->
   <xacro:unless value="${color == 'none'}">
@@ -43,127 +45,13 @@
     <origin rpy="0.000000 0.000000 0.000000" xyz="0.000000 1.175000 0.000000"/>
   </joint>
-  <!-- TORRE DE HANOI -->
-  <link name="hanoi_base">
-    <visual>
-      <origin xyz="-0.058 -0.044 -0.01" rpy="0 0 0" />
-      <geometry>
-        <mesh filename="package://tm_description/meshes/hanoi/base.stl" scale="0.001 0.001 0.001"/>
-      </geometry>
-      <material name="Color_hbase">
-        <color rgba="0.643 0.454 0.286 1"/>
-      </material>
-    </visual>
-  </link>
-  <!-- arrumar medidas do robo esq para pino1 da torre -->
-  <joint name="Jmesa" type="fixed">
-    <origin xyz="0.3 0.4 0" rpy="0 0 1.57" />
+  <joint name="base_to_left1" type="fixed">
     <parent link="base"/>
-    <child link="hanoi_base"/>
+    <child link="left1base"/>
+    <origin rpy="0.000000 0.000000 0.000000" xyz="-1.000000 0.000000 0.000000"/>
   </joint>
-  <joint name="Jp1" type="prismatic">
-    <origin xyz="0 0 0" rpy="0 0 0" />
-    <limit effort="30" velocity="1.0" lower="-2.2" upper="0.7" />
-    <parent link="hanoi_base"/>
-    <child link="hanoi_p1"/>
-  </joint>
-  <link name="hanoi_p1">
-    <visual>
-      <origin xyz="0 0 0" rpy="0 0 0" />
-      <geometry>
-        <mesh filename="package://tm_description/meshes/hanoi/peca_vermelha_1.stl" scale="0.001 0.001 0.001"/>
-      </geometry>
-      <!--material name="Peca_amarela">
-        <color rgba="1 0.788 0.121 1"/-->
-      <!--material name="Peca_azul">
-        <color rgba="0 0.352 0.580 1"/-->
-      <material name="Peca_vermelha">
-        <color rgba="0.901 0.168 0.156 1"/>
-      </material>
-    </visual>
-  </link>
-  <link name="hanoi_p2">
-    <visual>
-      <origin xyz="0 0 0" rpy="0 0 0" />
-      <geometry>
-        <mesh filename="package://tm_description/meshes/hanoi/peca_vermelha_2.stl" scale="0.001 0.001 0.001"/>
-      </geometry>
-      <material name="Peca_vermelha">
-        <color rgba="0.901 0.168 0.156 1"/>
-      </material>
-    </visual>
-  </link>
-  <joint name="Jp2" type="prismatic">
-    <origin xyz="0 0 0.013" rpy="0 0 0" />
-    <limit effort="30" velocity="1.0" lower="-2.2" upper="0.7" />
-    <parent link="hanoi_base"/>
-    <child link="hanoi_p2"/>
-  </joint>
-  <link name="hanoi_p3">
-    <visual>
-      <origin xyz="0 0 0" rpy="0 0 0" />
-      <geometry>
-        <mesh filename="package://tm_description/meshes/hanoi/peca_vermelha_3.stl" scale="0.001 0.001 0.001"/>
-      </geometry>
-      <material name="Peca_vermelha">
-        <color rgba="0.901 0.168 0.156 1"/>
-      </material>
-    </visual>
-  </link>
-  <joint name="Jp3" type="prismatic">
-    <origin xyz="0 0 0.026" rpy="0 0 0" />
-    <limit effort="30" velocity="1.0" lower="-2.2" upper="0.7" />
-    <parent link="hanoi_base"/>
-    <child link="hanoi_p3"/>
-  </joint>
-  <link name="hanoi_p4">
-    <visual>
-      <origin xyz="0 0 0" rpy="0 0 0" />
-      <geometry>
-        <mesh filename="package://tm_description/meshes/hanoi/peca_verde_1.stl" scale="0.001 0.001 0.001"/>
-      </geometry>
-      <material name="Peca_verde">
-        <color rgba="0.670 0.858 0.160 1"/>
-      </material>
-    </visual>
-  </link>
-  <joint name="Jp4" type="prismatic">
-    <origin xyz="0.088 0 0" rpy="0 0 0" />
-    <limit effort="30" velocity="1.0" lower="-2.2" upper="0.7" />
-    <parent link="hanoi_base"/>
-    <child link="hanoi_p4"/>
-  </joint>
-  <link name="hanoi_p5">
-    <visual>
-      <origin xyz="0 0 0" rpy="0 0 0" />
-      <geometry>
-        <mesh filename="package://tm_description/meshes/hanoi/peca_verde_2.stl" scale="0.001 0.001 0.001"/>
-      </geometry>
-      <material name="Peca_verde">
-        <color rgba="0.670 0.858 0.160 1"/>
-      </material>
-    </visual>
-  </link>
-  <joint name="Jp5" type="prismatic">
-    <origin xyz="0.088 0 0.013" rpy="0 0 0" />
-    <limit effort="30" velocity="1.0" lower="-2.2" upper="0.7" />
-    <parent link="hanoi_base"/>
-    <child link="hanoi_p5"/>
-  </joint>
-  <link name="hanoi_p6">
-    <visual>
-      <origin xyz="0 0 0" rpy="0 0 0" />
-      <geometry>
-        <mesh filename="package://tm_description/meshes/hanoi/peca_verde_3.stl" scale="0.001 0.001 0.001"/>
-      </geometry>
-      <material name="Peca_verde">
-        <color rgba="0.670 0.858 0.160 1"/>
-      </material>
-    </visual>
-  </link>
-  <joint name="Jp6" type="prismatic">
-    <origin xyz="0.088 0 0.026" rpy="0 0 0" />
-    <limit effort="30" velocity="1.0" lower="-2.2" upper="0.7" />
-    <parent link="hanoi_base"/>
-    <child link="hanoi_p6"/>
+  <joint name="base_to_right1" type="fixed">
+    <parent link="base"/>
+    <child link="right1base"/>
+    <origin rpy="0.000000 0.000000 0.000000" xyz="-1.000000 1.175000 0.000000"/>
   </joint>
 </robot>

Commit message: modified:   Comandos.txt 	modified:   tm_description/xacro/tm5-700.urdf.xacro

File: tm_description/xacro/tm5-700.urdf.xacro (robot description, xacro)
@@ -27,4 +27,6 @@
   <xacro:tm5-700 ns="$(arg ns)" prefix="left1" color="green" format="stl"/>
   <xacro:tm5-700 ns="$(arg ns)" prefix="right1" color="green" format="stl"/>
+  <xacro:tm5-700 ns="$(arg ns)" prefix="left2" color="yellow" format="stl"/>
+  <xacro:tm5-700 ns="$(arg ns)" prefix="right2" color="yellow" format="stl"/>
   <!-- Arm.color.stl -->
   <xacro:unless value="${color == 'none'}">
@@ -48,10 +50,20 @@
     <parent link="base"/>
     <child link="left1base"/>
-    <origin rpy="0.000000 0.000000 0.000000" xyz="-1.000000 0.000000 0.000000"/>
+    <origin rpy="0.000000 0.000000 0.000000" xyz="-1.500000 0.000000 0.000000"/>
   </joint>
   <joint name="base_to_right1" type="fixed">
     <parent link="base"/>
     <child link="right1base"/>
-    <origin rpy="0.000000 0.000000 0.000000" xyz="-1.000000 1.175000 0.000000"/>
+    <origin rpy="0.000000 0.000000 0.000000" xyz="-1.500000 1.175000 0.000000"/>
+  </joint>
+  <joint name="base_to_left2" type="fixed">
+    <parent link="base"/>
+    <child link="left2base"/>
+    <origin rpy="0.000000 0.000000 0.000000" xyz="-3.000000 0.000000 0.000000"/>
+  </joint>
+  <joint name="base_to_right2" type="fixed">
+    <parent link="base"/>
+    <child link="right2base"/>
+    <origin rpy="0.000000 0.000000 0.000000" xyz="-3.000000 1.175000 0.000000"/>
   </joint>
 </robot>
