Commit message: modified:   tm_description/urdf/tm5700.urdf

File: tm_description/urdf/tm5700.urdf (robot description, URDF)
Before this commit: robot tm5-700, 19 links, 18 joints
Links:
- link leftlink_0: geometry collision mesh filename=/home/piatan/tmdriver_ws/src/tm_description/meshes/tm5-900/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; visual mesh filename=/home/piatan/tmdriver_ws/src/tm_description/meshes/tm5-900/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
- link leftlink_1: geometry collision mesh filename=/home/piatan/tmdriver_ws/src/tm_description/meshes/tm5-900/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; visual mesh filename=/home/piatan/tmdriver_ws/src/tm_description/meshes/tm5-900/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
- link leftlink_2: geometry collision mesh filename=/home/piatan/tmdriver_ws/src/tm_description/meshes/tm5-700/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; visual mesh filename=/home/piatan/tmdriver_ws/src/tm_description/meshes/tm5-700/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
- link leftlink_3: geometry collision mesh filename=/home/piatan/tmdriver_ws/src/tm_description/meshes/tm5-700/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; visual mesh filename=/home/piatan/tmdriver_ws/src/tm_description/meshes/tm5-700/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
- link leftlink_4: geometry collision mesh filename=/home/piatan/tmdriver_ws/src/tm_description/meshes/tm5-900/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; visual mesh filename=/home/piatan/tmdriver_ws/src/tm_description/meshes/tm5-900/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
- link leftlink_5: geometry collision mesh filename=/home/piatan/tmdriver_ws/src/tm_description/meshes/tm5-900/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; visual mesh filename=/home/piatan/tmdriver_ws/src/tm_description/meshes/tm5-900/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
- link leftlink_6: geometry collision mesh filename=/home/piatan/tmdriver_ws/src/tm_description/meshes/tm5-900/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; visual mesh filename=/home/piatan/tmdriver_ws/src/tm_description/meshes/tm5-900/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
- link rightlink_0: geometry collision mesh filename=/home/piatan/tmdriver_ws/src/tm_description/meshes/tm5-900/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; visual mesh filename=/home/piatan/tmdriver_ws/src/tm_description/meshes/tm5-900/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
- link rightlink_1: geometry collision mesh filename=/home/piatan/tmdriver_ws/src/tm_description/meshes/tm5-900/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; visual mesh filename=/home/piatan/tmdriver_ws/src/tm_description/meshes/tm5-900/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
- link rightlink_2: geometry collision mesh filename=/home/piatan/tmdriver_ws/src/tm_description/meshes/tm5-700/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; visual mesh filename=/home/piatan/tmdriver_ws/src/tm_description/meshes/tm5-700/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
- link rightlink_3: geometry collision mesh filename=/home/piatan/tmdriver_ws/src/tm_description/meshes/tm5-700/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; visual mesh filename=/home/piatan/tmdriver_ws/src/tm_description/meshes/tm5-700/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
- link rightlink_4: geometry collision mesh filename=/home/piatan/tmdriver_ws/src/tm_description/meshes/tm5-900/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; visual mesh filename=/home/piatan/tmdriver_ws/src/tm_description/meshes/tm5-900/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
- link rightlink_5: geometry collision mesh filename=/home/piatan/tmdriver_ws/src/tm_description/meshes/tm5-900/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; visual mesh filename=/home/piatan/tmdriver_ws/src/tm_description/meshes/tm5-900/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
- link rightlink_6: geometry collision mesh filename=/home/piatan/tmdriver_ws/src/tm_description/meshes/tm5-900/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; visual mesh filename=/home/piatan/tmdriver_ws/src/tm_description/meshes/tm5-900/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
